Commit message: robot moving with teleop

File: description/robot.urdf.xacro (robot description, xacro)
@@ -2,3 +2,4 @@
 <robot xmlns:xacro="http://www.ros.org/wiki/xacro"  name="robot">
     <xacro:include filename="robot_core.xacro"/>
+    <xacro:include filename="gazebo_control.xacro"/>
 </robot>

File: description/robot_core.xacro (robot description, xacro)
@@ -44,7 +44,7 @@
         </xacro:inertial_box>
     </link>
-    <!-- <gazebo reference="chassis">
+    <gazebo reference="chassis">
         <material>Gazebo/Orange</material>
-    </gazebo> -->
+    </gazebo>
     <!-- LEFT WHEEL LINK -->
     <joint name="left_wheel_joint" type="continuous">
@@ -70,7 +70,7 @@
         </xacro:inertial_cylinder>
     </link>
-    <!-- <gazebo reference="left_wheel">
+    <gazebo reference="left_wheel">
         <material>Gazebo/Blue</material>
-    </gazebo> -->
+    </gazebo>
     <!-- RIGHT WHEEL LINK -->
     <joint name="right_wheel_joint" type="continuous">
@@ -96,7 +96,7 @@
         </xacro:inertial_cylinder>
     </link>
-    <!-- <gazebo reference="right_wheel">
+    <gazebo reference="right_wheel">
         <material>Gazebo/Blue</material>
-    </gazebo> -->
+    </gazebo>
         <!-- CASTER WHEEL LINK -->
     <joint name="caster_wheel_joint" type="fixed">
@@ -121,3 +121,8 @@
         </xacro:inertial_sphere>
     </link>
+    <gazebo reference="caster_wheel">
+        <material>Gazebo/Black</material>
+        <mu1 value="0.001"/>
+        <mu2 value="0.001"/>
+    </gazebo>
 </robot>
